File: JFP_board_v2.kicad_sch (KiCad schematic)
At the start: 81 parts, among them J1 SPI2 external, J2 RX header, J3 I2C2 external, J4 UART4 external, J5 SWD conn, J6 ESC conn, J7 918-418K2023S40001, Q1 AO3400A, SW1 BOOT0, U1 TPS5430DDAR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

Commit message: Added HP203B pressure sensor
Parts:
- added C20: 4.7uF, Capacitor_SMD:C_0603_1608Metric, symbol Device:C_Small
- added U7: HP203B, _custom_footprints:LGA-8_3.6x3.8x0.9P, symbol _custom_symbols:HP203B
- R10, R23, R24: footprint Capacitor_SMD:C_0402_1005Metric -> Resistor_SMD:R_0402_1005Metric
Connections:
- net +3V3: now also C20.1, U7.3 (VDD), U7.8 (CSB)
- net GND: now also C20.2, U7.2 (GND)
- net I2C2_SCL: now also U7.5 (SCL)
- net I2C2_SDA: now also U7.6 (SDA)
- net HP203B_INT1: now reaches U3.37 (PC6)
- net HP203B_INT1: now also U7.1 (INT1)
Other:
- note added: "Pressure"
- moved on the sheet: JP1, Q1, R21, R22

Commit message: Production files
Parts:
- J7: LCSC C167321 -> C709357
Other:
- title: JFP board v2 -> Quad board v2
Changed lines of the file:
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@@
   (paper "A3")
   (title_block
-    (title "JFP board v2")
+    (title "Quad board v2")
     (date "2022-12-28")
     (rev "1")
@@
       (effects (font (size 1.27 1.27)) hide)
     )
-    (property "LCSC" "C167321" (id 4) (at 29.21 207.01 0))
+    (property "LCSC" "C709357" (id 4) (at 29.21 207.01 0))
     (pin "A1")
     (pin "A12")
